Commit message: 第七章：机器人导航

File: ROS_demo/demo03_ws/src/two_urdf02_gazebo/urdf/demo02_car_base.urdf.xacro (robot description, xacro)
@@ -93,5 +93,5 @@
         </gazebo>
         <!-- 3.2、joint -->
-        <joint name="${wheel_name}2link" type="continuous">
+        <joint name="${wheel_name}_wheel_joint" type="continuous"> <!--修改处2023/11/16-->
             <parent link="base_link"/>
             <child link="${wheel_name}_wheel"/>
@@ -105,6 +105,6 @@
         </joint>
     </xacro:macro>
-    <xacro:wheel_func wheel_name="left" flag="1" />
-    <xacro:wheel_func wheel_name="right" flag="-1" />
+    <xacro:wheel_func wheel_name="base_l" flag="1" />
+    <xacro:wheel_func wheel_name="base_r" flag="-1" />
     <!-- 4、添加万象轮 -->
     <!--

File: ROS_demo/demo03_ws/src/two_urdf02_gazebo/urdf/gazebo/move.xacro (robot description, xacro)
@@ -21,13 +21,13 @@
         <plugin name="differential_drive_controller" filename="libgazebo_ros_diff_drive.so">
             <rosDebugLevel>Debug</rosDebugLevel>
-            <publishWheelTF>true</publishWheelTF>
+            <publishWheelTF>false</publishWheelTF> <!--修改警告添加：2023/11/16-->
             <robotNamespace>/</robotNamespace>
             <publishTf>1</publishTf>
-            <publishWheelJointState>true</publishWheelJointState>
+            <publishWheelJointState>false</publishWheelJointState>
             <alwaysOn>true</alwaysOn>
-            <updateRate>100.0</updateRate>
+            <updateRate>10.0</updateRate>     <!-- 修改警告添加：2023/11/16、但未实际运行也可以：另一修改在launch文件夹的demo03_env.launch-->
             <legacyMode>true</legacyMode>
-            <leftJoint>left2link</leftJoint> <!-- 左轮 -->
-            <rightJoint>right2link</rightJoint> <!-- 右轮 -->
+            <leftJoint>base_l_wheel_joint</leftJoint> <!-- 左轮 -->
+            <rightJoint>base_r_wheel_joint</rightJoint> <!-- 右轮 -->
             <wheelSeparation>${base_radius * 2}</wheelSeparation> <!-- 车轮间距 -->
             <wheelDiameter>${wheel_radius * 2}</wheelDiameter> <!-- 车轮直径 -->
